Commit message: fix robot model launch file and urdf

File: descriptions/material.xacro (robot description, xacro)
@@ -1,9 +1,9 @@
 <?xml version="1.0" ?>
 <robot xmlns:xacro="http://www.ros.org/wiki/xacro">
-  <material name="white">
-    <color rgba="1 1 1 1"/>
+  <material name="base_link">
+    <color rgba="0.9 0.1 0.9 1.0" />
   </material>
   <material name="black">
-    <color rgba="1 1 1 1"/>
+    <color rgba="0.1 0.1 0.1 1.0" />
   </material>
   <material name="red">

File: descriptions/robot_core.xacro (robot description, xacro)
@@ -1,5 +1,4 @@
 <?xml version="1.0" ?>
 <robot xmlns:xacro="http://www.ros.org/wiki/xacro">
-  <xacro:include filename="material.xacro" />
   <!-- base link -->
   <link name="base_link">
@@ -9,5 +8,5 @@
         <box size="0.27 0.185 0.055" />
       </geometry>
-      <material name="white" />
+      <material name="base_link" />
     </visual>
   </link>

File: descriptions/sensor.xacro (robot description, xacro)
@@ -1,8 +1,7 @@
 <?xml version="1.0" ?>
 <robot xmlns:xacro="http://www.ros.org/wiki/xacro">
-  <xacro:include filename="material.xacro" />
   <!-- laser -->
   <joint name="laser_joint" type="fixed">
-    <origin xyz="0.06 0.00 0.20" rpy="0 0 ${pi/2}" />
+    <origin xyz="0.05 0.00 0.18" rpy="0 0 ${pi/2}" />
     <parent link="base_link" />
     <child link="laser_link" />
@@ -12,5 +11,5 @@
       <origin xyz="0 0 0" rpy="0 0 0" />
       <geometry>
-        <cylinder radius="0.04" length="0.03" />
+        <cylinder radius="0.03" length="0.02" />
       </geometry>
       <material name="red" />
@@ -19,5 +18,5 @@
   <!-- gyro -->
   <joint name="gyro_joint" type="fixed">
-    <origin xyz="0 0 0" rpy="0 0 0" />
+    <origin xyz="-0.04 0.00 0.14" rpy="0 0 0" />
     <parent link="base_link" />
     <child link="gyro_link" />

File: descriptions/wheeltec.urdf.xacro (robot description, xacro)
@@ -1,5 +1,5 @@
 <?xml version="1.0" ?>
 <robot xmlns:xacro="http://www.ros.org/wiki/xacro" name="wheeltec">
-  <xacro:arg name="sim_mode" default="false"/>
+  <xacro:include filename="material.xacro" />
   <xacro:include filename="robot_core.xacro" />
   <xacro:include filename="sensor.xacro" />
