Commit message: WIP: description files for gazebo

File: descriptions/wheeltec/material.xacro (robot description, xacro)
@@ -1,5 +1,5 @@
 <?xml version="1.0" ?>
 <robot xmlns:xacro="http://www.ros.org/wiki/xacro">
-  <material name="base_link">
+  <material name="purple">
     <color rgba="0.9 0.1 0.9 1.0" />
   </material>

File: descriptions/wheeltec/robot_core.xacro (robot description, xacro)
@@ -1,16 +1,57 @@
-<?xml version="1.0" ?>
+<?xml version="1.0"?>
 <robot xmlns:xacro="http://www.ros.org/wiki/xacro">
+  <xacro:include filename="inertial_macros.xacro"/>
+  <material name="purple">
+    <color rgba="0.9 0.1 0.9 1.0" />
+  </material>
+  <material name="black">
+    <color rgba="0.1 0.1 0.1 1.0" />
+  </material>
+  <material name="red">
+    <color rgba="1 0.1 0.1 1" />
+  </material>
+  <material name="orange">
+    <color rgba="1 0.55 0 1" />
+  </material>
   <!-- base link -->
   <link name="base_link">
+  </link>
+  <!-- base_footprint link -->
+  <joint name="base_footprint_joint" type="fixed">
+    <parent link="base_link"/>
+    <child link="base_footprint"/>
+    <origin xyz="0 0 0" rpy="0 0 0"/>
+  </joint>
+  <link name="base_footprint">
+  </link>
+  <!-- chassis link -->
+  <joint name="chassis_joint" type="fixed">
+    <parent link="base_link"/>
+    <child link="chassis"/>
+    <origin xyz="-0.2 0 0.0975"/>
+  </joint>
+  <link name="base_link">
     <visual>
-      <origin xyz="0 0 0.0975" rpy="0 0 0" />
+      <origin xyz="0.135 0 0.0275" />
       <geometry>
         <box size="0.27 0.185 0.055" />
       </geometry>
-      <material name="base_link" />
+      <material name="purple" />
     </visual>
+    <collision>
+      <origin xyz="0.135 0 0.0275"/>
+      <geometry>
+        <box size="0.27 0.185 0.055"/>
+      </geometry>
+    </collision>
+    <xacro:inertial_box mass="0.5" x="0.27" y="0.185" z="0.055">
+      <origin xyz="0.135 0 0.0275" rpy="0 0 0"/>
+    </xacro:inertial_box>
   </link>
+  <gazebo reference="chassis">
+    <material>Gazebo/Purple</material>
+  </gazebo>
   <!-- left rear wheel -->
-  <joint name="left_wheel_joint" type="continuous">
+  <!-- <joint name="left_wheel_joint" type="continuous">
     <origin xyz="-0.085 0.0975 0.0375" rpy="${pi/2} 0 0" />
     <parent link="base_link" />
@@ -26,7 +67,7 @@
       <material name="black" />
     </visual>
-  </link>
+  </link> -->
   <!-- right rear wheel -->
-  <joint name="right_wheel_joint" type="continuous">
+  <!-- <joint name="right_wheel_joint" type="continuous">
     <origin xyz="-0.085 -0.0975 0.0375" rpy="${pi/2} 0 0" />
     <parent link="base_link" />
@@ -42,7 +83,7 @@
       <material name="black" />
     </visual>
-  </link>
+  </link> -->
   <!-- left front wheel -->
-  <joint name="left_front_joint" type="continuous">
+  <!-- <joint name="left_front_joint" type="continuous">
     <origin xyz="0.085 0.0975 0.0375" rpy="${pi/2} 0 0" />
     <parent link="base_link" />
@@ -58,7 +99,7 @@
       <material name="black" />
     </visual>
-  </link>
+  </link> -->
   <!-- right front wheel -->
-  <joint name="right_front_joint" type="continuous">
+  <!-- <joint name="right_front_joint" type="continuous">
     <origin xyz="0.085 -0.0975 0.0375" rpy="${pi/2} 0 0" />
     <parent link="base_link" />
@@ -74,4 +115,4 @@
       <material name="black" />
     </visual>
-  </link>
+  </link> -->
 </robot>
