Commit message: finish fixing urdf description files

File: descriptions/wheeltec/robot_core.xacro (robot description, xacro)
@@ -2,16 +2,4 @@
 <robot xmlns:xacro="http://www.ros.org/wiki/xacro">
   <xacro:include filename="inertial_macros.xacro"/>
-  <material name="purple">
-    <color rgba="0.9 0.1 0.9 1.0" />
-  </material>
-  <material name="black">
-    <color rgba="0.1 0.1 0.1 1.0" />
-  </material>
-  <material name="red">
-    <color rgba="1 0.1 0.1 1" />
-  </material>
-  <material name="orange">
-    <color rgba="1 0.55 0 1" />
-  </material>
   <!-- base link -->
   <link name="base_link">
@@ -29,9 +17,9 @@
     <parent link="base_link"/>
     <child link="chassis"/>
-    <origin xyz="-0.2 0 0.0975"/>
+    <origin xyz="0 0 0.0975"/>
   </joint>
-  <link name="base_link">
+  <link name="chassis">
     <visual>
-      <origin xyz="0.135 0 0.0275" />
+      <origin xyz="0 0 0" />
       <geometry>
         <box size="0.27 0.185 0.055" />
@@ -40,5 +28,5 @@
     </visual>
     <collision>
-      <origin xyz="0.135 0 0.0275"/>
+      <origin xyz="0 0 0"/>
       <geometry>
         <box size="0.27 0.185 0.055"/>
@@ -46,5 +34,5 @@
     </collision>
     <xacro:inertial_box mass="0.5" x="0.27" y="0.185" z="0.055">
-      <origin xyz="0.135 0 0.0275" rpy="0 0 0"/>
+      <origin xyz="0 0 0" rpy="0 0 0"/>
     </xacro:inertial_box>
   </link>
@@ -53,9 +41,9 @@
   </gazebo>
   <!-- left rear wheel -->
-  <!-- <joint name="left_wheel_joint" type="continuous">
-    <origin xyz="-0.085 0.0975 0.0375" rpy="${pi/2} 0 0" />
+  <joint name="left_wheel_joint" type="continuous">
+    <origin xyz="-0.085 0.0975 0.0375" rpy="-${pi/2} 0 0" />
     <parent link="base_link" />
     <child link="left_wheel_link" />
-    <axis xyz="0 1 0" />
+    <axis xyz="0 0 1" />
   </joint>
   <link name="left_wheel_link">
@@ -67,11 +55,22 @@
       <material name="black" />
     </visual>
-  </link> -->
+    <collision>
+      <geometry>
+        <cylinder radius="0.0375" length="0.03" />
+      </geometry>
+    </collision>
+    <xacro:inertial_cylinder mass="0.1" length="0.03" radius="0.0375">
+      <origin xyz="0 0 0" rpy="0 0 0"/>
+    </xacro:inertial_cylinder>
+  </link>
+  <gazebo reference="left_wheel_link">
+    <material>Gazebo/Black</material>
+  </gazebo>
   <!-- right rear wheel -->
-  <!-- <joint name="right_wheel_joint" type="continuous">
+  <joint name="right_wheel_joint" type="continuous">
     <origin xyz="-0.085 -0.0975 0.0375" rpy="${pi/2} 0 0" />
     <parent link="base_link" />
     <child link="right_wheel_link" />
-    <axis xyz="0 1 0" />
+    <axis xyz="0 0 -1" />
   </joint>
   <link name="right_wheel_link">
@@ -83,11 +82,22 @@
       <material name="black" />
     </visual>
-  </link> -->
+    <collision>
+      <geometry>
+        <cylinder radius="0.0375" length="0.03" />
+      </geometry>
+    </collision>
+    <xacro:inertial_cylinder mass="0.1" length="0.03" radius="0.0375">
+      <origin xyz="0 0 0" rpy="0 0 0"/>
+    </xacro:inertial_cylinder>
+  </link>
+  <gazebo reference="right_wheel_link">
+    <material>Gazebo/Black</material>
+  </gazebo>
   <!-- left front wheel -->
-  <!-- <joint name="left_front_joint" type="continuous">
-    <origin xyz="0.085 0.0975 0.0375" rpy="${pi/2} 0 0" />
+  <joint name="left_front_joint" type="continuous">
+    <origin xyz="0.085 0.0975 0.0375" rpy="-${pi/2} 0 0" />
     <parent link="base_link" />
     <child link="left_front_link" />
-    <axis xyz="0 1 0" />
+    <axis xyz="0 0 1" />
   </joint>
   <link name="left_front_link">
@@ -99,11 +109,22 @@
       <material name="black" />
     </visual>
-  </link> -->
+    <collision>
+      <geometry>
+        <cylinder radius="0.0375" length="0.03" />
+      </geometry>
+    </collision>
+    <xacro:inertial_cylinder mass="0.1" length="0.03" radius="0.0375">
+      <origin xyz="0 0 0" rpy="0 0 0"/>
+    </xacro:inertial_cylinder>
+  </link>
+  <gazebo reference="left_front_link">
+    <material>Gazebo/Black</material>
+  </gazebo>
   <!-- right front wheel -->
-  <!-- <joint name="right_front_joint" type="continuous">
+  <joint name="right_front_joint" type="continuous">
     <origin xyz="0.085 -0.0975 0.0375" rpy="${pi/2} 0 0" />
     <parent link="base_link" />
     <child link="right_front_link" />
-    <axis xyz="0 1 0" />
+    <axis xyz="0 0 -1" />
   </joint>
   <link name="right_front_link">
@@ -115,4 +136,15 @@
       <material name="black" />
     </visual>
-  </link> -->
+    <collision>
+      <geometry>
+        <cylinder radius="0.0375" length="0.03" />
+      </geometry>
+    </collision>
+    <xacro:inertial_cylinder mass="0.1" length="0.03" radius="0.0375">
+      <origin xyz="0 0 0" rpy="0 0 0"/>
+    </xacro:inertial_cylinder>
+  </link>
+  <gazebo reference="right_front_link">
+    <material>Gazebo/Black</material>
+  </gazebo>
 </robot>

File: descriptions/wheeltec/sensor.xacro (robot description, xacro)
@@ -16,4 +16,7 @@
     </visual>
   </link>
+  <gazebo reference="laser_link">
+    <material>Gazebo/Red</material>
+  </gazebo>
   <!-- gyro -->
   <joint name="gyro_joint" type="fixed">
@@ -24,10 +27,13 @@
   <link name="gyro_link">
     <visual>
-    <origin xyz="0 0 0" rpy="0 0 0" />
-    <geometry>
-      <box size="0.04 0.03 0.015" />
-    </geometry>
-    <material name="orange" />
+      <origin xyz="0 0 0" rpy="0 0 0" />
+      <geometry>
+        <box size="0.04 0.03 0.015" />
+      </geometry>
+      <material name="orange" />
     </visual>
   </link>
+  <gazebo reference="gyro_link">
+    <material>Gazebo/Orange</material>
+  </gazebo>
 </robot>

File: descriptions/wheeltec/wheeltec.urdf.xacro (robot description, xacro)
@@ -1,6 +1,6 @@
 <?xml version="1.0"?>
 <robot xmlns:xacro="http://www.ros.org/wiki/xacro" name="wheeltec">
-  <!-- <xacro:include filename="material.xacro" /> -->
+  <xacro:include filename="material.xacro" />
   <xacro:include filename="robot_core.xacro" />
-  <!-- <xacro:include filename="sensor.xacro" /> -->
+  <xacro:include filename="sensor.xacro" />
 </robot>

Commit message: change wheel joints to fixed to resolve transforms not found issue

File: descriptions/wheeltec/robot_core.xacro (robot description, xacro)
@@ -41,5 +41,5 @@
   </gazebo>
   <!-- left rear wheel -->
-  <joint name="left_wheel_joint" type="continuous">
+  <joint name="left_wheel_joint" type="fixed">
     <origin xyz="-0.085 0.0975 0.0375" rpy="-${pi/2} 0 0" />
     <parent link="base_link" />
@@ -68,5 +68,5 @@
   </gazebo>
   <!-- right rear wheel -->
-  <joint name="right_wheel_joint" type="continuous">
+  <joint name="right_wheel_joint" type="fixed">
     <origin xyz="-0.085 -0.0975 0.0375" rpy="${pi/2} 0 0" />
     <parent link="base_link" />
@@ -95,5 +95,5 @@
   </gazebo>
   <!-- left front wheel -->
-  <joint name="left_front_joint" type="continuous">
+  <joint name="left_front_joint" type="fixed">
     <origin xyz="0.085 0.0975 0.0375" rpy="-${pi/2} 0 0" />
     <parent link="base_link" />
@@ -122,5 +122,5 @@
   </gazebo>
   <!-- right front wheel -->
-  <joint name="right_front_joint" type="continuous">
+  <joint name="right_front_joint" type="fixed">
     <origin xyz="0.085 -0.0975 0.0375" rpy="${pi/2} 0 0" />
     <parent link="base_link" />
