Commit message: modify robot description files, and slam launch to incorporate namespace for nodes, topics, and tf frames

File: descriptions/wheeltec/gazebo_control.xacro (robot description, xacro)
@@ -5,7 +5,7 @@
       <commandTopic>cmd_vel</commandTopic>
       <odometryTopic>odom</odometryTopic>
-      <odometryFrame>odom</odometryFrame>
+      <odometryFrame>$(arg namespace)/odom</odometryFrame>
       <odometryRate>20.0</odometryRate>
-      <robotBaseFrame>base_link</robotBaseFrame>
+      <robotBaseFrame>$(arg namespace)/base_link</robotBaseFrame>
       <cmdTimeout>0.5</cmdTimeout>
     </plugin>

File: descriptions/wheeltec/robot_core.xacro (robot description, xacro)
@@ -3,21 +3,19 @@
   <xacro:include filename="inertial_macros.xacro"/>
   <!-- base link -->
-  <link name="base_link">
-  </link>
+  <link name="$(arg namespace)/base_link" />
   <!-- base_footprint link -->
-  <joint name="base_footprint_joint" type="fixed">
-    <parent link="base_link"/>
-    <child link="base_footprint"/>
+  <joint name="$(arg namespace)/base_footprint_joint" type="fixed">
+    <parent link="$(arg namespace)/base_link"/>
+    <child link="$(arg namespace)/base_footprint"/>
     <origin xyz="0 0 0" rpy="0 0 0"/>
   </joint>
-  <link name="base_footprint">
-  </link>
+  <link name="$(arg namespace)/base_footprint" />
   <!-- chassis link -->
-  <joint name="chassis_joint" type="fixed">
-    <parent link="base_link"/>
-    <child link="chassis"/>
+  <joint name="$(arg namespace)/chassis_joint" type="fixed">
+    <parent link="$(arg namespace)/base_link"/>
+    <child link="$(arg namespace)/chassis"/>
     <origin xyz="0 0 0.0975"/>
   </joint>
-  <link name="chassis">
+  <link name="$(arg namespace)/chassis">
     <visual>
       <origin xyz="0 0 0" />
@@ -37,15 +35,15 @@
     </xacro:inertial_box>
   </link>
-  <gazebo reference="chassis">
+  <gazebo reference="$(arg namespace)/chassis">
     <material>Gazebo/Purple</material>
   </gazebo>
   <!-- left rear wheel -->
-  <joint name="left_wheel_joint" type="fixed">
+  <joint name="$(arg namespace)/left_wheel_joint" type="fixed">
     <origin xyz="-0.085 0.0975 0.0375" rpy="-${pi/2} 0 0" />
-    <parent link="base_link" />
-    <child link="left_wheel_link" />
+    <parent link="$(arg namespace)/base_link" />
+    <child link="$(arg namespace)/left_wheel_link" />
     <axis xyz="0 0 1" />
   </joint>
-  <link name="left_wheel_link">
+  <link name="$(arg namespace)/left_wheel_link">
     <visual>
       <origin xyz="0 0 0" rpy="0 0 0" />
@@ -64,15 +62,15 @@
     </xacro:inertial_cylinder>
   </link>
-  <gazebo reference="left_wheel_link">
+  <gazebo reference="$(arg namespace)/left_wheel_link">
     <material>Gazebo/Black</material>
   </gazebo>
   <!-- right rear wheel -->
-  <joint name="right_wheel_joint" type="fixed">
+  <joint name="$(arg namespace)/right_wheel_joint" type="fixed">
     <origin xyz="-0.085 -0.0975 0.0375" rpy="${pi/2} 0 0" />
-    <parent link="base_link" />
-    <child link="right_wheel_link" />
+    <parent link="$(arg namespace)/base_link" />
+    <child link="$(arg namespace)/right_wheel_link" />
     <axis xyz="0 0 -1" />
   </joint>
-  <link name="right_wheel_link">
+  <link name="$(arg namespace)/right_wheel_link">
     <visual>
       <origin xyz="0 0 0" rpy="0 0 0" />
@@ -91,15 +89,15 @@
     </xacro:inertial_cylinder>
   </link>
-  <gazebo reference="right_wheel_link">
+  <gazebo reference="$(arg namespace)/right_wheel_link">
     <material>Gazebo/Black</material>
   </gazebo>
   <!-- left front wheel -->
-  <joint name="left_front_joint" type="fixed">
+  <joint name="$(arg namespace)/left_front_joint" type="fixed">
     <origin xyz="0.085 0.0975 0.0375" rpy="-${pi/2} 0 0" />
-    <parent link="base_link" />
-    <child link="left_front_link" />
+    <parent link="$(arg namespace)/base_link" />
+    <child link="$(arg namespace)/left_front_link" />
     <axis xyz="0 0 1" />
   </joint>
-  <link name="left_front_link">
+  <link name="$(arg namespace)/left_front_link">
     <visual>
       <origin xyz="0 0 0" rpy="0 0 0" />
@@ -118,15 +116,15 @@
     </xacro:inertial_cylinder>
   </link>
-  <gazebo reference="left_front_link">
+  <gazebo reference="$(arg namespace)/left_front_link">
     <material>Gazebo/Black</material>
   </gazebo>
   <!-- right front wheel -->
-  <joint name="right_front_joint" type="fixed">
+  <joint name="$(arg namespace)/right_front_joint" type="fixed">
     <origin xyz="0.085 -0.0975 0.0375" rpy="${pi/2} 0 0" />
-    <parent link="base_link" />
-    <child link="right_front_link" />
+    <parent link="$(arg namespace)/base_link" />
+    <child link="$(arg namespace)/right_front_link" />
     <axis xyz="0 0 -1" />
   </joint>
-  <link name="right_front_link">
+  <link name="$(arg namespace)/right_front_link">
     <visual>
       <origin xyz="0 0 0" rpy="0 0 0" />
@@ -145,5 +143,5 @@
     </xacro:inertial_cylinder>
   </link>
-  <gazebo reference="right_front_link">
+  <gazebo reference="$(arg namespace)/right_front_link">
     <material>Gazebo/Black</material>
   </gazebo>

File: descriptions/wheeltec/sensor.xacro (robot description, xacro)
@@ -2,10 +2,10 @@
 <robot xmlns:xacro="http://www.ros.org/wiki/xacro">
   <!-- laser -->
-  <joint name="laser_joint" type="fixed">
+  <joint name="$(arg namespace)/laser_joint" type="fixed">
     <origin xyz="0.05 0.00 0.18" rpy="0 0 0" />
-    <parent link="base_link" />
-    <child link="laser_link" />
+    <parent link="$(arg namespace)/base_link" />
+    <child link="$(arg namespace)/laser_link" />
   </joint>
-  <link name="laser_link">
+  <link name="$(arg namespace)/laser_link">
     <visual>
       <origin xyz="0 0 0" rpy="0 0 0" />
@@ -16,5 +16,5 @@
     </visual>
   </link>
-  <gazebo reference="laser_link">
+  <gazebo reference="$(arg namespace)/laser_link">
     <material>Gazebo/Red</material>
     <sensor name="laser" type="ray">
@@ -42,17 +42,17 @@
         </noise>
       </ray>
-      <plugin name="laser_controller" filename="libgazebo_ros_laser.so">
-        <topicName>/scan</topicName>
-        <frameName>laser_link</frameName>
+      <plugin name="$(arg namespace)/laser" filename="libgazebo_ros_laser.so">
+        <topicName>scan</topicName>
+        <frameName>$(arg namespace)/laser_link</frameName>
       </plugin>
     </sensor>
   </gazebo>
   <!-- gyro -->
-  <joint name="gyro_joint" type="fixed">
+  <joint name="$(arg namespace)/gyro_joint" type="fixed">
     <origin xyz="-0.04 0.00 0.14" rpy="0 0 0" />
-    <parent link="base_link" />
-    <child link="gyro_link" />
+    <parent link="$(arg namespace)/base_link" />
+    <child link="$(arg namespace)/gyro_link" />
   </joint>
-  <link name="gyro_link">
+  <link name="$(arg namespace)/gyro_link">
     <visual>
       <origin xyz="0 0 0" rpy="0 0 0" />
@@ -63,5 +63,5 @@
     </visual>
   </link>
-  <gazebo reference="gyro_link">
+  <gazebo reference="$(arg namespace)/gyro_link">
     <material>Gazebo/Orange</material>
   </gazebo>

File: descriptions/wheeltec/wheeltec.urdf.xacro (robot description, xacro)
@@ -1,4 +1,5 @@
 <?xml version="1.0"?>
 <robot xmlns:xacro="http://www.ros.org/wiki/xacro" name="wheeltec">
+  <xacro:arg name="namespace" default="robot" />
   <xacro:include filename="material.xacro" />
   <xacro:include filename="robot_core.xacro" />
