Commit message: setup for multiple robots (#5)
* modify robot description files, and slam launch to incorporate namespace for nodes, topics, and tf frames

* modify navigation launch file and params to use robot namespace

* create willow garage gazebo world, and spawn robot there

* create turtlebot house world

* adjust sensor and navigation capabilities for a larger and more open environment

* generate 2 turtlebot house maps

* fix gazebo and navigation launch files

* create sim_multi launch file and rviz config

* update rrt_exploration_multi rviz config

* tune navigation parameters

* update rrt_exploration_multi rviz config

* generate multirobot maps for turtlebot_stage4

File: descriptions/wheeltec/sensor.xacro (robot description, xacro)
@@ -2,10 +2,10 @@
 <robot xmlns:xacro="http://www.ros.org/wiki/xacro">
   <!-- laser -->
-  <joint name="laser_joint" type="fixed">
+  <joint name="$(arg namespace)/laser_joint" type="fixed">
     <origin xyz="0.05 0.00 0.18" rpy="0 0 0" />
-    <parent link="base_link" />
-    <child link="laser_link" />
+    <parent link="$(arg namespace)/base_link" />
+    <child link="$(arg namespace)/laser_link" />
   </joint>
-  <link name="laser_link">
+  <link name="$(arg namespace)/laser_link">
     <visual>
       <origin xyz="0 0 0" rpy="0 0 0" />
@@ -16,5 +16,5 @@
     </visual>
   </link>
-  <gazebo reference="laser_link">
+  <gazebo reference="$(arg namespace)/laser_link">
     <material>Gazebo/Red</material>
     <sensor name="laser" type="ray">
@@ -33,5 +33,5 @@
         <range>
           <min>0.05</min>
-          <max>3</max>
+          <max>12</max>
           <resolution>0.005</resolution>
         </range>
@@ -42,17 +42,17 @@
         </noise>
       </ray>
-      <plugin name="laser_controller" filename="libgazebo_ros_laser.so">
-        <topicName>/scan</topicName>
-        <frameName>laser_link</frameName>
+      <plugin name="$(arg namespace)/laser" filename="libgazebo_ros_laser.so">
+        <topicName>scan</topicName>
+        <frameName>$(arg namespace)/laser_link</frameName>
       </plugin>
     </sensor>
   </gazebo>
   <!-- gyro -->
-  <joint name="gyro_joint" type="fixed">
+  <joint name="$(arg namespace)/gyro_joint" type="fixed">
     <origin xyz="-0.04 0.00 0.14" rpy="0 0 0" />
-    <parent link="base_link" />
-    <child link="gyro_link" />
+    <parent link="$(arg namespace)/base_link" />
+    <child link="$(arg namespace)/gyro_link" />
   </joint>
-  <link name="gyro_link">
+  <link name="$(arg namespace)/gyro_link">
     <visual>
       <origin xyz="0 0 0" rpy="0 0 0" />
@@ -63,5 +63,5 @@
     </visual>
   </link>
-  <gazebo reference="gyro_link">
+  <gazebo reference="$(arg namespace)/gyro_link">
     <material>Gazebo/Orange</material>
   </gazebo>
