Commit message: add laser sensors to wheeltec and articubot
spawn in turtlebot3_stage4 world

File: descriptions/articubot/robot.urdf.xacro (robot description, xacro)
@@ -10,5 +10,5 @@
         <xacro:include filename="gazebo_control.xacro" />
     <!-- </xacro:unless> -->
-    <!-- <xacro:include filename="lidar.xacro" /> -->
+    <xacro:include filename="lidar.xacro" />
     <!-- <xacro:include filename="camera.xacro" /> -->
     <!-- <xacro:include filename="depth_camera.xacro" /> -->

File: descriptions/wheeltec/sensor.xacro (robot description, xacro)
@@ -3,5 +3,5 @@
   <!-- laser -->
   <joint name="laser_joint" type="fixed">
-    <origin xyz="0.05 0.00 0.18" rpy="0 0 ${pi/2}" />
+    <origin xyz="0.05 0.00 0.18" rpy="0 0 0" />
     <parent link="base_link" />
     <child link="laser_link" />
@@ -18,4 +18,28 @@
   <gazebo reference="laser_link">
     <material>Gazebo/Red</material>
+    <sensor name="laser" type="ray">
+      <pose>0 0 0 0 0 0</pose>
+      <visualize>false</visualize>
+      <update_rate>10</update_rate>
+      <ray>
+        <scan>
+          <horizontal>
+            <samples>360</samples>
+            <resolution>1</resolution>
+            <min_angle>-3.14</min_angle>
+            <max_angle>3.14</max_angle>
+          </horizontal>
+        </scan>
+        <range>
+          <min>0.1</min>
+          <max>12</max>
+          <resolution>0.01</resolution>
+        </range>
+      </ray>
+      <plugin name="laser_controller" filename="libgazebo_ros_laser.so">
+        <topicName>/scan</topicName>
+        <frameName>laser_link</frameName>
+      </plugin>
+    </sensor>
   </gazebo>
   <!-- gyro -->
